Commit message: Made the cleats weightless in the urdf file experimenting with physics

File: resources/assets/bez/model/soccerbot_box_no_cleats.urdf (robot description, URDF)
Before this commit: robot soccerbot, 29 links, 28 joints
Links:
- removed link /left_foot_cleat_4
- removed link /left_foot_cleat_5
- removed link /left_foot_cleat_6
- removed link /left_foot_cleat_7
- removed link /right_foot_cleat_0
- removed link /right_foot_cleat_1
- removed link /right_foot_cleat_2
- removed link /right_foot_cleat_3
Joints:
- removed joint /left_foot_cleat_4
- removed joint /left_foot_cleat_5
- removed joint /left_foot_cleat_6
- removed joint /left_foot_cleat_7
- removed joint right_foot_cleat_0
- removed joint right_foot_cleat_1
- removed joint right_foot_cleat_2
- removed joint right_foot_cleat_3
