Commit message: Updated .dae files Created a new hybrid model with .dae files Modified yaml files Fixed a simulation breaking bug that caused improper reset of simulation

File: resources/assets/bez/model/soccerbot_stl.urdf (robot description, URDF)
Before this commit: robot soccerbot, 21 links, 20 joints
Links:
- link /head: geometry collision mesh filename=../meshes/head.dae scale=1 1 1; visual mesh filename=../meshes/head.dae scale=1 1 1
- link /left_ankle: geometry collision box size=0.090769 0.042 0.0506; visual mesh filename=../meshes/left_ankle.dae scale=1 1 1
- link /left_bicep: geometry collision mesh filename=../meshes/left_bicep.dae scale=1 1 1; visual mesh filename=../meshes/left_bicep.dae scale=1 1 1
- link /left_calve: geometry collision box size=0.031883 0.048 0.105683; visual mesh filename=../meshes/left_calve.dae scale=1 1 1
- link /left_foot: geometry collision box size=0.09 0.07 0.003; visual mesh filename=../meshes/left_foot.dae scale=1 1 1
- link /left_forearm: geometry collision mesh filename=../meshes/left_forearm.dae scale=1 1 1; visual mesh filename=../meshes/left_forearm.dae scale=1 1 1
- link /left_hip_front: geometry collision box size=0.083747 0.04885 0.0506; visual mesh filename=../meshes/left_hip_front.dae scale=1 1 1
- link /left_hip_side: geometry collision box size=0.0485 0.022 0.00005; visual mesh filename=../meshes/left_hip_side.dae scale=1 1 1
- link /left_thigh: geometry collision box size=0.022 0.048 0.111; visual mesh filename=../meshes/left_thigh.dae scale=1 1 1
- link /neck: geometry collision mesh filename=../meshes/neck.dae scale=1 1 1; visual mesh filename=../meshes/neck.dae scale=1 1 1
- link /right_ankle: geometry collision box size=0.090769 0.042 0.0506; visual mesh filename=../meshes/right_ankle.dae scale=1 1 1
- link /right_bicep: geometry collision mesh filename=../meshes/right_bicep.dae scale=1 1 1; visual mesh filename=../meshes/right_bicep.dae scale=1 1 1
- link /right_calve: geometry collision box size=0.031883 0.048 0.105683; visual mesh filename=../meshes/right_calve.dae scale=1 1 1
- link /right_foot: geometry collision box size=0.09 0.07 0.003; visual mesh filename=../meshes/right_foot.dae scale=1 1 1
- link /right_forearm: geometry collision mesh filename=../meshes/right_forearm.dae scale=1 1 1; visual mesh filename=../meshes/right_forearm.dae scale=1 1 1
- link /right_hip_front: geometry collision box size=0.083747 0.04885 0.0506; visual mesh filename=../meshes/right_hip_front.dae scale=1 1 1
- link /right_hip_side: geometry collision box size=0.0485 0.022 0.00005; visual mesh filename=../meshes/right_hip_side.dae scale=1 1 1
- link /right_thigh: geometry collision box size=0.022 0.048 0.111; visual mesh filename=../meshes/right_thigh.dae scale=1 1 1
- link /torso: geometry collision mesh filename=../meshes/torso.dae scale=1 1 1; visual mesh filename=../meshes/torso.dae scale=1 1 1
Joints:
- joint left_leg_motor_3: origin xyz=0 0 -0.0890 rpy=0 0 0 -> xyz=0 0 -0.08900 rpy=0 0 0
- joint left_leg_motor_4: origin xyz=0 0 -0.0827 rpy=0 0 0 -> xyz=0 0 -0.0865 rpy=0 0 0
- joint right_leg_motor_3: origin xyz=0 0 -0.0890 rpy=0 0 0 -> xyz=0 0 -0.089 rpy=0 0 0
- joint right_leg_motor_4: origin xyz=0 0 -0.0827 rpy=0 0 0 -> xyz=0 0 -0.0865 rpy=0 0 0
