Commit message: Added test_motor_action_agent to one by one rotate each motor Fixed a bug that would interfer with the reset procedure Added framework for torque control Experimented with parameter for optimal physics setting Renamed files to better represent the task

File: resources/assets/bez/model/soccerbot_box.urdf (robot description, URDF)
Before this commit: robot soccerbot, 21 links, 20 joints
Links:
- link /left_bicep: mass 0.213e-3 -> 0.000213

Commit message: Found issues in self collision Edit leg motors collision boxes. DOF 7/ Left_leg_motor_3 collision box might be too big

File: resources/assets/bez/model/soccerbot_box.urdf (robot description, URDF)
Before this commit: robot soccerbot, 21 links, 20 joints
Links:
- link /left_foot: geometry collision box size=0.09 0.07 0.00674; visual box size=0.09 0.07 0.00674
- link /right_foot: geometry collision box size=0.09 0.07 0.00674; visual box size=0.09 0.07 0.00674

Commit message: Added cleats to feet. Finished foot pressure sensors function Imported observation function

File: resources/assets/bez/model/soccerbot_box.urdf (robot description, URDF)
Before this commit: robot soccerbot, 21 links, 20 joints
Links:
- added link /left_foot_cleat_4, mass 23.216e-3; collision box size=0.01 0.01 0.002; visual box size=0.01 0.01 0.002
- added link /left_foot_cleat_5, mass 23.216e-3; collision box size=0.01 0.01 0.002; visual box size=0.01 0.01 0.002
- added link /left_foot_cleat_6, mass 23.216e-3; collision box size=0.01 0.01 0.002; visual box size=0.01 0.01 0.002
- added link /left_foot_cleat_7, mass 23.216e-3; collision box size=0.01 0.01 0.002; visual box size=0.01 0.01 0.002
- added link /right_foot_cleat_0, mass 23.216e-3; collision box size=0.01 0.01 0.002; visual box size=0.01 0.01 0.002
- added link /right_foot_cleat_1, mass 23.216e-3; collision box size=0.01 0.01 0.002; visual box size=0.01 0.01 0.002
- added link /right_foot_cleat_2, mass 23.216e-3; collision box size=0.01 0.01 0.002; visual box size=0.01 0.01 0.002
- added link /right_foot_cleat_3, mass 23.216e-3; collision box size=0.01 0.01 0.002; visual box size=0.01 0.01 0.002
Joints:
- added joint /left_foot_cleat_4: type fixed, parent /left_foot, child /left_foot_cleat_4, origin xyz=0.0 0 0.0 rpy=0 0 0, axis 0 0 0
- added joint /left_foot_cleat_5: type fixed, parent /left_foot, child /left_foot_cleat_5, origin xyz=0.0 0 0.0 rpy=0 0 0, axis 0 0 0
- added joint /left_foot_cleat_6: type fixed, parent /left_foot, child /left_foot_cleat_6, origin xyz=0.0 0 0.0 rpy=0 0 0, axis 0 0 0
- added joint /left_foot_cleat_7: type fixed, parent /left_foot, child /left_foot_cleat_7, origin xyz=0.0 0 0.0 rpy=0 0 0, axis 0 0 0
- added joint right_foot_cleat_0: type fixed, parent /right_foot, child /right_foot_cleat_0, origin xyz=0.0 0 0.0 rpy=0 0 0, axis 0 0 0
- added joint right_foot_cleat_1: type fixed, parent /right_foot, child /right_foot_cleat_1, origin xyz=0.0 0 0.0 rpy=0 0 0, axis 0 0 0
- added joint right_foot_cleat_2: type fixed, parent /right_foot, child /right_foot_cleat_2, origin xyz=0.0 0 0.0 rpy=0 0 0, axis 0 0 0
- added joint right_foot_cleat_3: type fixed, parent /right_foot, child /right_foot_cleat_3, origin xyz=0.0 0 0.0 rpy=0 0 0, axis 0 0 0

Commit message: Optimized calculations (imu, off_orn, feet) by converting them to torch.jit.script Implemented foot pressure sensors for no cleats Tuned hyperparameter Renamed models to stay in convention Added feet pressure sensors to reward function for increased stabilization

File: resources/assets/bez/model/soccerbot_box.urdf (robot description, URDF)
Before this commit: robot soccerbot, 29 links, 28 joints
Links:
- removed link /left_foot_cleat_4
- removed link /left_foot_cleat_5
- removed link /left_foot_cleat_6
- removed link /left_foot_cleat_7
- removed link /right_foot_cleat_0
- removed link /right_foot_cleat_1
- removed link /right_foot_cleat_2
- removed link /right_foot_cleat_3
Joints:
- removed joint /left_foot_cleat_4
- removed joint /left_foot_cleat_5
- removed joint /left_foot_cleat_6
- removed joint /left_foot_cleat_7
- removed joint right_foot_cleat_0
- removed joint right_foot_cleat_1
- removed joint right_foot_cleat_2
- removed joint right_foot_cleat_3
- joint right_leg_motor_4: origin xyz=0 0 -0.0827 rpy=0 0 0 -> xyz=0 0 -0.0865 rpy=0 0 0

File: resources/assets/bez/model/soccerbot_box_sensor.urdf (robot description, URDF)
Before this commit: robot soccerbot, 21 links, 20 joints
Links:
- added link /left_foot_cleat_4, mass 5e-3; collision box size=0.01 0.01 0.002; visual box size=0.01 0.01 0.002
- added link /left_foot_cleat_5, mass 5e-3; collision box size=0.01 0.01 0.002; visual box size=0.01 0.01 0.002
- added link /left_foot_cleat_6, mass 5e-3; collision box size=0.01 0.01 0.002; visual box size=0.01 0.01 0.002
- added link /left_foot_cleat_7, mass 5e-3; collision box size=0.01 0.01 0.002; visual box size=0.01 0.01 0.002
- added link /right_foot_cleat_0, mass 5e-3; collision box size=0.01 0.01 0.002; visual box size=0.01 0.01 0.002
- added link /right_foot_cleat_1, mass 5e-3; collision box size=0.01 0.01 0.002; visual box size=0.01 0.01 0.002
- added link /right_foot_cleat_2, mass 5e-3; collision box size=0.01 0.01 0.002; visual box size=0.01 0.01 0.002
- added link /right_foot_cleat_3, mass 5e-3; collision box size=0.01 0.01 0.002; visual box size=0.01 0.01 0.002
Joints:
- added joint /left_foot_cleat_4: type fixed, parent /left_foot, child /left_foot_cleat_4, origin xyz=0.0 0 0.0 rpy=0 0 0, axis 0 0 0
- added joint /left_foot_cleat_5: type fixed, parent /left_foot, child /left_foot_cleat_5, origin xyz=0.0 0 0.0 rpy=0 0 0, axis 0 0 0
- added joint /left_foot_cleat_6: type fixed, parent /left_foot, child /left_foot_cleat_6, origin xyz=0.0 0 0.0 rpy=0 0 0, axis 0 0 0
- added joint /left_foot_cleat_7: type fixed, parent /left_foot, child /left_foot_cleat_7, origin xyz=0.0 0 0.0 rpy=0 0 0, axis 0 0 0
- added joint right_foot_cleat_0: type fixed, parent /right_foot, child /right_foot_cleat_0, origin xyz=0.0 0 0.0 rpy=0 0 0, axis 0 0 0
- added joint right_foot_cleat_1: type fixed, parent /right_foot, child /right_foot_cleat_1, origin xyz=0.0 0 0.0 rpy=0 0 0, axis 0 0 0
- added joint right_foot_cleat_2: type fixed, parent /right_foot, child /right_foot_cleat_2, origin xyz=0.0 0 0.0 rpy=0 0 0, axis 0 0 0
- added joint right_foot_cleat_3: type fixed, parent /right_foot, child /right_foot_cleat_3, origin xyz=0.0 0 0.0 rpy=0 0 0, axis 0 0 0
- joint right_leg_motor_4: origin xyz=0 0 -0.0865 rpy=0 0 0 -> xyz=0 0 -0.0827 rpy=0 0 0
